File: IO_16x8_matrix/IO_16x8_matrix.kicad_pcb (KiCad board)
At the start: 2 copper layers, 97.6 x 67.3 mm, 173 parts, among them J1 Conn_01x06, J2 nmount SW Debug, J3 USB_C_Receptacle_USB2.0, J4 Conn_01x06, J6 Conn_01x10, J7 Conn_01x09, J8 Conn_01x12, J9 nmount TPs, Q1 2N7002, Q10 AO3401A, Q11 AO3401A, Q12 AO3401A, Q13 2N7002, Q14 2N7002, Q15 AO3401A, Q16 AO3401A, Q17 AO3400A, Q18 AO3400A, Q19 AO3400A, Q2 2N7002, Q20 AO3400A, Q21 AO3400A, Q22 AO3400A, Q23 AO3400A, Q24 AO3400A, Q25 AO3400A, Q26 AO3400A, Q3 2N7002, Q4 AO3401A, Q5 AO3401A, Q6 AO3401A, Q7 2N7002, Q8 2N7002, Q9 2N7002, SW1 Reset, SW2 Boot, SW3 ADDRESS, U1 ADM3483, U10 L78L24_SOT89, U11 L78L24_SOT89, U12 L78L24_SOT89, U13 L78L24_SOT89, U14 LMV321, U2 W25Q128JVSIQ, U3 RP2040, U4 SN74AHCT1G125, U5 AP2112K-3.3, U6 L78L24_SOT89, U7 L78L24_SOT89, U8 L78L24_SOT89, U9 L78L24_SOT89, Y1 12MHz,18pF

Commit message: routed
Parts:
- removed Q10, Q11, Q12, Q15, Q16: AO3401A, Package_TO_SOT_SMD:SOT-23
- removed Q13, Q14, Q9: 2N7002, Package_TO_SOT_SMD:SOT-23
- removed Q17, Q18, Q19, Q20, Q21, Q22, Q23, Q24, Q25, Q26: AO3400A, Package_TO_SOT_SMD:SOT-23
- removed the REF** at (108.2, 49.7)
- removed the REF** at (150.6, 106.4)
- removed the REF** at (190.0, 49.8)
- removed TP1: TP_IO26, TestPoint:TestPoint_Pad_D1.0mm
- removed TP2, TP8: TP_IO27, TestPoint:TestPoint_Pad_D1.0mm
- removed U10, U11, U12, U13: L78L24_SOT89, Package_TO_SOT_SMD:SOT-89-3
- added C43: 100n, Capacitor_SMD:C_0402_1005Metric, F.Cu at (115.1, 72.3)
- added C44: 100n, Capacitor_SMD:C_0402_1005Metric, F.Cu at (119.6, 69.2)
- added C45: 100n, Capacitor_SMD:C_0402_1005Metric, F.Cu at (115.1, 75.2)
- added C46: 100n, Capacitor_SMD:C_0402_1005Metric, F.Cu at (115.1, 77.3)
- added C47: 100n, Capacitor_SMD:C_0402_1005Metric, F.Cu at (122.2, 79.4)
- added C48: 100n, Capacitor_SMD:C_0402_1005Metric, F.Cu at (115.1, 80.4)
- added C49: 100n, Capacitor_SMD:C_0402_1005Metric, F.Cu at (115.1, 82.3)
- added C50: 100n, Capacitor_SMD:C_0402_1005Metric, F.Cu at (119.6, 79.4)
- added C51: 100n, Capacitor_SMD:C_0402_1005Metric, F.Cu at (115.1, 85.5)
- added C52: 100n, Capacitor_SMD:C_0402_1005Metric, F.Cu at (115.1, 87.6)
- added C53: 100n, Capacitor_SMD:C_0402_1005Metric, F.Cu at (122.2, 89.4)
- added C54: 100n, Capacitor_SMD:C_0402_1005Metric, F.Cu at (115.1, 89.8)
- added C55: 100n, Capacitor_SMD:C_0402_1005Metric, F.Cu at (115.1, 91.7)
- added C56: 100n, Capacitor_SMD:C_0402_1005Metric, F.Cu at (119.6, 89.4)
- added C57: 100n, Capacitor_SMD:C_0402_1005Metric, F.Cu at (115.1, 95.4)
- added C58: 100n, Capacitor_SMD:C_0402_1005Metric, F.Cu at (115.1, 97.5)
- added D10: 1N4148WS, Diode_SMD:D_SOD-323, F.Cu at (106.7, 66.4)
- added D11: 1N4148WS, Diode_SMD:D_SOD-323, F.Cu at (106.7, 70.1)
- added D12: 1N4148WS, Diode_SMD:D_SOD-323, F.Cu at (106.7, 72.1)
- added D13: 1N4148WS, Diode_SMD:D_SOD-323, F.Cu at (106.7, 74.1)
- added D14: 1N4148WS, Diode_SMD:D_SOD-323, F.Cu at (106.7, 76.2)
- added D15: 1N4148WS, Diode_SMD:D_SOD-323, F.Cu at (106.8, 79.8)
- added D16: 1N4148WS, Diode_SMD:D_SOD-323, F.Cu at (106.8, 81.8)
- added D17: 1N4148WS, Diode_SMD:D_SOD-323, F.Cu at (106.8, 83.8)
- added D18: 1N4148WS, Diode_SMD:D_SOD-323, F.Cu at (106.8, 85.9)
- added D19: 1N4148WS, Diode_SMD:D_SOD-323, F.Cu at (107.4, 88.5)
- added D20: 1N4148WS, Diode_SMD:D_SOD-323, F.Cu at (107.4, 91.8)
- added D21: 1N4148WS, Diode_SMD:D_SOD-323, F.Cu at (107.4, 95.4)
- added D22: 1N4148WS, Diode_SMD:D_SOD-323, F.Cu at (108.1, 98.0)
- added D7: 1N4148WS, Diode_SMD:D_SOD-323, F.Cu at (106.7, 60.3)
- added D8: 1N4148WS, Diode_SMD:D_SOD-323, F.Cu at (106.7, 62.3)
- added D9: 1N4148WS, Diode_SMD:D_SOD-323, F.Cu at (106.7, 64.4)
- added J5: Conn_01x09, Connector_Molex:Molex_KK-254_AE-6410-09A_1x09_P2.54mm_Vertical, F.Cu at (195.6, 82.5)
- added R65: 10k, Resistor_SMD:R_0603_1608Metric, F.Cu at (126.6, 73.8)
- added R66: 10k, Resistor_SMD:R_0603_1608Metric, F.Cu at (126.6, 75.6)
- added R67: 100R, Resistor_SMD:R_0603_1608Metric, F.Cu at (112.9, 74.3)
- added R68: 100R, Resistor_SMD:R_0603_1608Metric, F.Cu at (112.9, 76.3)
- added R69: 1k, Resistor_SMD:R_0603_1608Metric, F.Cu at (109.9, 74.3)
- added R70: 1k, Resistor_SMD:R_0603_1608Metric, F.Cu at (109.9, 76.3)
- added R71: 10k, Resistor_SMD:R_0603_1608Metric, F.Cu at (126.0, 78.6)
- added R72: 10k, Resistor_SMD:R_0603_1608Metric, F.Cu at (126.0, 81.7)
- added R73: 100R, Resistor_SMD:R_0603_1608Metric, F.Cu at (113.0, 80.1)
- added R74: 100R, Resistor_SMD:R_0603_1608Metric, F.Cu at (113.0, 82.4)
- added R75: 1k, Resistor_SMD:R_0603_1608Metric, F.Cu at (110.0, 80.1)
- added R76: 1k, Resistor_SMD:R_0603_1608Metric, F.Cu at (110.0, 81.8)
- added R77: 10k, Resistor_SMD:R_0603_1608Metric, F.Cu at (126.0, 84.7)
- added R78: 10k, Resistor_SMD:R_0603_1608Metric, F.Cu at (126.0, 87.8)
- added R79: 100R, Resistor_SMD:R_0603_1608Metric, F.Cu at (113.0, 84.6)
- added R80: 100R, Resistor_SMD:R_0603_1608Metric, F.Cu at (113.0, 86.7)
- added R81: 1k, Resistor_SMD:R_0603_1608Metric, F.Cu at (110.0, 84.6)
- added R82: 1k, Resistor_SMD:R_0603_1608Metric, F.Cu at (110.0, 86.2)
- added R83: 10k, Resistor_SMD:R_0603_1608Metric, F.Cu at (126.7, 90.4)
- added R84: 10k, Resistor_SMD:R_0603_1608Metric, F.Cu at (126.7, 92.1)
- added R85: 100R, Resistor_SMD:R_0603_1608Metric, F.Cu at (113.0, 89.4)
- added R86: 100R, Resistor_SMD:R_0603_1608Metric, F.Cu at (113.0, 91.6)
- added R87: 1k, Resistor_SMD:R_0603_1608Metric, F.Cu at (110.0, 89.4)
- added R88: 1k, Resistor_SMD:R_0603_1608Metric, F.Cu at (110.0, 91.2)
- added R89: 10k, Resistor_SMD:R_0603_1608Metric, F.Cu at (126.7, 96.5)
- added R90: 10k, Resistor_SMD:R_0603_1608Metric, F.Cu at (126.7, 94.6)
- added R91: 100R, Resistor_SMD:R_0603_1608Metric, F.Cu at (113.0, 94.0)
- added R92: 100R, Resistor_SMD:R_0603_1608Metric, F.Cu at (113.0, 96.3)
- added R93: 1k, Resistor_SMD:R_0603_1608Metric, F.Cu at (110.0, 94.0)
- added R94: 1k, Resistor_SMD:R_0603_1608Metric, F.Cu at (110.0, 96.0)
- added REF**: MountingHole_5.5mm_Pinball, IO_16x8_matrix:MountingHole_5.5mm_Pinball, F.Cu at (150.6, 106.4)
- added REF**: MountingHole_5.5mm_Pinball, IO_16x8_matrix:MountingHole_5.5mm_Pinball, F.Cu at (108.2, 49.8)
- added REF**: MountingHole_5.5mm_Pinball, IO_16x8_matrix:MountingHole_5.5mm_Pinball, F.Cu at (190.0, 49.8)
- C25, C26, C27, C28, C29, C30, C31, C32: value 1u 50V -> 10n
- C33: value 1u 50V -> 10u
- C34, C35, C36, C37, C38, C39, C40: value 1u 50V -> 100n; footprint Capacitor_SMD:C_0603_1608Metric -> Capacitor_SMD:C_0402_1005Metric
- C41: value 100µ 35V -> 100n; footprint Capacitor_SMD:CP_Elec_6.3x7.7 -> Capacitor_SMD:C_0402_1005Metric
- J6: value Conn_01x10 -> Conn_01x09; footprint Connector_Molex:Molex_KK-396_5273-10A_1x10_P3.96mm_Vertical -> Connector_Molex:Molex_KK-396_5273-09A_1x09_P3.96mm_Vertical
- J8: value Conn_01x12 -> Conn_01x10; footprint Connector_Molex:Molex_KK-396_5273-12A_1x12_P3.96mm_Vertical -> Connector_Molex:Molex_KK-396_5273-10A_1x10_P3.96mm_Vertical
- J9: value nmount TPs -> Conn_01x10; footprint Connector_PinSocket_2.54mm:PinSocket_1x03_P2.54mm_Vertical -> Connector_Molex:Molex_KK-396_5273-10A_1x10_P3.96mm_Vertical
- Q1, Q2, Q3, Q7, Q8: value 2N7002 -> MMBT3904
- Q4, Q5, Q6: value AO3401A -> MMBT3904
- R20, R21, R22, R26, R27, R28, R32, R33: value 2k -> 1k
- R23, R24, R25, R29, R30, R31, R34, R35: value 3k3 -> 1k
- R36, R37: value 10k -> 2k
- R42, R43, R48, R49, R54, R55: value 100R -> 1k
- R46, R47, R52, R53: value 10k -> 100R
- R50, R51: value 100R -> 10k
- U6, U7, U8, U9: value L78L24_SOT89 -> LM339; footprint Package_TO_SOT_SMD:SOT-89-3 -> Package_SO:SOIC-14_3.9x8.7mm_P1.27mm
- moved C41 75.6 mm to (115.1, 70.4), turned to -90 degrees
- moved C39 74.2 mm to (115.1, 66.9), turned to -90 degrees
- moved C36 72.8 mm to (115.1, 62.4), turned to -90 degrees
- moved C33 72.2 mm to (112.3, 57.7), turned to 90 degrees
- moved C35 70.5 mm to (115.1, 60.1), turned to -90 degrees
- moved C37 69.2 mm to (119.8, 59.4)
- moved C34 61.4 mm to (122.0, 59.4), turned to 0 degrees
- moved J9 59.9 mm to (194.3, 105.4), turned to 180 degrees
- moved C38 56.4 mm to (115.1, 64.6), turned to -90 degrees
- moved U6 55.1 mm to (120.3, 63.8), turned to -90 degrees
- moved U8 55.1 mm to (120.3, 83.8), turned to -90 degrees
- moved U9 54.3 mm to (120.3, 93.9), turned to -90 degrees
- moved U7 53.7 mm to (120.3, 73.7), turned to -90 degrees
- moved C40 53.6 mm to (122.2, 69.2), turned to 0 degrees
- moved SW3 49.7 mm to (174.8, 90.8)
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Connections:
- C25 pad 1: /20V -> /Driver8/D1
- C26 pad 1: /20V -> /Driver8/D2
- C27 pad 1: /20V -> /Driver8/D3
- C28 pad 1: Net-(C28-Pad1) -> /Driver8/D4
- C29 pad 1: Net-(C29-Pad1) -> /Driver8/D5
- C30 pad 1: Net-(C30-Pad1) -> /Driver8/D6
- C31 pad 1: /20V -> /Driver8/D7
- C32 pad 1: /20V -> /Driver8/D8
- C33 pad 1: /20V -> /In16/V_SWITCH
- C34 pad 1: Net-(C34-Pad1) -> +5V
- C37 pad 1: /20V -> /In16/V_SWITCH
- C38 pad 1: /20V -> Net-(C38-Pad1)
- C40 pad 1: Net-(C40-Pad1) -> +5V
- C41 pad 1: /20V -> Net-(C41-Pad1)
- J4 pad 1: /20V -> /5V_IN
- J6 pad 1: /Hi8/H1 -> /Driver8/D1
- J6 pad 3: /Hi8/H2 -> /Driver8/D2
- J6 pad 4: /Hi8/H3 -> /Driver8/D3
- J6 pad 5: /Hi8/H4 -> /Driver8/D4
- J6 pad 6: /Hi8/H5 -> /Driver8/D5
- J6 pad 7: /Hi8/H6 -> /Driver8/D6
- J6 pad 8: /Hi8/H7 -> /Driver8/D7
- J6 pad 9: /Hi8/H8 -> /Driver8/D8
- J7 pad 1: /Lo10/L1 -> /In16/T1
- J7 pad 2: /Lo10/L2 -> /In16/T2
- J7 pad 3: unconnected-(J7-Pad3) -> /In16/T3
- J7 pad 4: /Lo10/L3 -> /In16/T4
- J7 pad 5: /Lo10/L4 -> /In16/T5
- J7 pad 6: /Lo10/L5 -> unconnected-(J7-Pad6)
- J7 pad 7: /Lo10/L6 -> /In16/T6
- J7 pad 8: /Lo10/L7 -> /In16/T7
- J7 pad 9: /Lo10/L8 -> /In16/T8
- J8 pad 1: /Lo10/L1 -> /In16/T8
- J8 pad 10: /Lo10/L9 -> unconnected-(J8-Pad10)
- J8 pad 2: /Lo10/L2 -> /In16/T7
- J8 pad 3: /Lo10/L3 -> /In16/T6
- J8 pad 4: /Lo10/L4 -> unconnected-(J8-Pad4)
- J8 pad 5: /Lo10/L5 -> /In16/T5
- J8 pad 6: /Lo10/L6 -> /In16/T4
- J8 pad 7: unconnected-(J8-Pad7) -> /In16/T3
- J8 pad 8: /Lo10/L7 -> /In16/T2
- J8 pad 9: /Lo10/L8 -> /In16/T1
- J9 pad 1: Net-(J9-Pad1) -> /In16/T16
- J9 pad 2: Net-(J9-Pad2) -> /In16/T15
- J9 pad 3: Net-(J9-Pad3) -> /In16/T14
- Q1 pad 1: /Hi_1 -> Net-(Q1-Pad1)
- Q1 pad 3: Net-(Q1-Pad3) -> /Driver8/D1
- Q2 pad 1: /Hi_3 -> Net-(Q2-Pad1)
- Q2 pad 3: Net-(Q2-Pad3) -> /Driver8/D2
- Q3 pad 1: /Hi_2 -> Net-(Q3-Pad1)
- Q3 pad 3: Net-(Q3-Pad3) -> /Driver8/D3
- Q4 pad 2: Net-(C28-Pad1) -> GND
- Q4 pad 3: /Hi8/H1 -> /Driver8/D4
- Q5 pad 2: Net-(C29-Pad1) -> GND
- Q5 pad 3: /Hi8/H3 -> /Driver8/D5
- Q6 pad 2: Net-(C30-Pad1) -> GND
- Q6 pad 3: /Hi8/H2 -> /Driver8/D6
- Q7 pad 1: /Hi_4 -> Net-(Q7-Pad1)
- Q7 pad 3: Net-(Q7-Pad3) -> /Driver8/D7
- Q8 pad 1: /Hi_5 -> Net-(Q8-Pad1)
- Q8 pad 3: Net-(Q8-Pad3) -> /Driver8/D8
- R20 pad 1: Net-(C28-Pad1) -> /Out_1
- R20 pad 2: Net-(Q4-Pad1) -> Net-(Q1-Pad1)
- R21 pad 1: Net-(C29-Pad1) -> /Out_2
- R21 pad 2: Net-(Q5-Pad1) -> Net-(Q2-Pad1)
- R22 pad 1: Net-(C30-Pad1) -> /Out_3
- R22 pad 2: Net-(Q6-Pad1) -> Net-(Q3-Pad1)
- R23 pad 1: Net-(Q4-Pad1) -> /Out_4
- R23 pad 2: Net-(Q1-Pad3) -> Net-(Q4-Pad1)
- R24 pad 1: Net-(Q5-Pad1) -> +5V
- R24 pad 2: Net-(Q2-Pad3) -> /Driver8/D1
- R25 pad 1: Net-(Q6-Pad1) -> +5V
- R25 pad 2: Net-(Q3-Pad3) -> /Driver8/D2
- R26 pad 1: Net-(C34-Pad1) -> +5V
- R26 pad 2: Net-(Q10-Pad1) -> /Driver8/D3
- R27 pad 1: Net-(C35-Pad1) -> +5V
- R27 pad 2: Net-(Q11-Pad1) -> /Driver8/D4
- R28 pad 1: Net-(C36-Pad1) -> /Out_5
- R28 pad 2: Net-(Q12-Pad1) -> Net-(Q5-Pad1)
- R29 pad 1: Net-(Q10-Pad1) -> /Out_6
- R29 pad 2: Net-(Q7-Pad3) -> Net-(Q6-Pad1)
- R30 pad 1: Net-(Q11-Pad1) -> /Out_7
- R30 pad 2: Net-(Q8-Pad3) -> Net-(Q7-Pad1)
- R31 pad 1: Net-(Q12-Pad1) -> /Out_8
- R31 pad 2: Net-(Q9-Pad3) -> Net-(Q8-Pad1)
- R32 pad 1: Net-(C39-Pad1) -> +5V
- R32 pad 2: Net-(Q15-Pad1) -> /Driver8/D5
- R33 pad 1: Net-(C40-Pad1) -> +5V
- R33 pad 2: Net-(Q16-Pad1) -> /Driver8/D6
- R34 pad 1: Net-(Q15-Pad1) -> +5V
- R34 pad 2: Net-(Q13-Pad3) -> /Driver8/D7
- R35 pad 1: Net-(Q16-Pad1) -> +5V
- R35 pad 2: Net-(Q14-Pad3) -> /Driver8/D8
- R36 pad 1: /Lo_1 -> +5V
- R36 pad 2: GND -> /In16/V_SWITCH
- R37 pad 1: /Lo_2 -> /In16/V_SWITCH
- R38 pad 1: /Lo_3 -> +3V3
- R38 pad 2: GND -> /In_1
- R39 pad 1: /Lo_4 -> +3V3
- R39 pad 2: GND -> /In_2
- R40 pad 1: /Lo_1 -> Net-(C35-Pad1)
- R40 pad 2: Net-(Q17-Pad1) -> Net-(D7-Pad2)
- R41 pad 1: /Lo_2 -> Net-(C36-Pad1)
- R41 pad 2: Net-(Q18-Pad1) -> Net-(D8-Pad2)
- R42 pad 1: /Lo_3 -> +5V
- R42 pad 2: Net-(Q19-Pad1) -> Net-(D7-Pad2)
- R43 pad 1: /Lo_4 -> +5V
- R43 pad 2: Net-(Q20-Pad1) -> Net-(D8-Pad2)
- R44 pad 1: /Lo_5 -> +3V3
- R44 pad 2: GND -> /In_3
- R45 pad 1: /Lo_6 -> +3V3
- R45 pad 2: GND -> /In_4
- R46 pad 1: /Lo_7 -> Net-(C38-Pad1)
- R46 pad 2: GND -> Net-(D9-Pad2)
- R47 pad 1: /Lo_8 -> Net-(C39-Pad1)
- R47 pad 2: GND -> Net-(D10-Pad2)
- R48 pad 1: /Lo_5 -> +5V
- R48 pad 2: Net-(Q21-Pad1) -> Net-(D9-Pad2)
- R49 pad 1: /Lo_6 -> +5V
- R49 pad 2: Net-(Q22-Pad1) -> Net-(D10-Pad2)
- R50 pad 1: /Lo_7 -> +3V3
- R50 pad 2: Net-(Q23-Pad1) -> /In_5
- R51 pad 1: /Lo_8 -> +3V3
- R51 pad 2: Net-(Q24-Pad1) -> /In_6
- R52 pad 1: /Lo_9 -> Net-(C41-Pad1)
- R52 pad 2: GND -> Net-(D11-Pad2)
- R53 pad 1: /Lo_10 -> Net-(C43-Pad1)
- R53 pad 2: GND -> Net-(D12-Pad2)
- R54 pad 1: /Lo_9 -> +5V
- R54 pad 2: Net-(Q25-Pad1) -> Net-(D11-Pad2)
- R55 pad 1: /Lo_10 -> +5V
- R55 pad 2: Net-(Q26-Pad1) -> Net-(D12-Pad2)
- U3 pad 11: /Lo_5 -> /In_6
- U3 pad 12: /Lo_4 -> /In_7
- U3 pad 13: /Lo_3 -> /In_8
- U3 pad 14: /Lo_2 -> /In_9
- U3 pad 15: /Lo_1 -> /In_10
- U3 pad 16: Net-(J9-Pad3) -> /In_11
- U3 pad 17: Net-(J9-Pad2) -> /In_12
- U3 pad 18: Net-(J9-Pad1) -> /In_13
- U3 pad 27: Net-(TP8-Pad1) -> /In_14
- U3 pad 28: /Hi_8 -> /In_15
- U3 pad 29: /Hi_7 -> /In_16
- U3 pad 30: /Hi_6 -> /Out_1
- U3 pad 31: /Hi_5 -> /Out_2
- U3 pad 32: /Hi_4 -> /Out_3
- U3 pad 34: /Hi_3 -> /Out_4
- U3 pad 35: /Hi_2 -> /Out_5
- U3 pad 36: /Hi_1 -> /Out_6
- U3 pad 38: Net-(TP1-Pad1) -> /Out_7
- U3 pad 39: Net-(TP2-Pad1) -> /Out_8
- U3 pad 5: /Lo_10 -> /In_1
- U3 pad 6: /Lo_9 -> /In_2
- U3 pad 7: /Lo_8 -> /In_3
- U3 pad 8: /Lo_7 -> /In_4
- U3 pad 9: /Lo_6 -> /In_5
- U6 pad 1: Net-(C28-Pad1) -> /In_2
- U6 pad 2: GND -> /In_1
- U6 pad 3: /20V -> +5V
- U7 pad 1: Net-(C29-Pad1) -> /In_6
- U7 pad 2: GND -> /In_5
- U7 pad 3: /20V -> +5V
- U8 pad 1: Net-(C30-Pad1) -> /In_10
- U8 pad 2: GND -> /In_9
- U8 pad 3: /20V -> +5V
- U9 pad 1: Net-(C34-Pad1) -> /In_14
- U9 pad 2: GND -> /In_13
- U9 pad 3: /20V -> +5V
Routing:
- net +5V: track 72.6 -> 297.3 mm, vias 5 -> 30
- net GND: track 190.8 -> 408.0 mm, vias 349 -> 339
- net /20V: track 113.9 -> 0.00 mm, vias 11 -> 0
- net /In16/V_SWITCH: track 0.00 -> 96.4 mm
- net /In16/T13: track 0.00 -> 94.1 mm
- net /In16/T16: track 0.00 -> 93.8 mm, vias 0 -> 1
- net /In16/T15: track 0.00 -> 93.6 mm, vias 0 -> 1
- net /In16/T14: track 0.00 -> 92.9 mm, vias 0 -> 1
- net /In16/T12: track 0.00 -> 89.2 mm
- net /In16/T11: track 0.00 -> 88.0 mm
- net /In16/T10: track 0.00 -> 86.4 mm
- net /In16/T9: track 0.00 -> 85.1 mm
- net +3V3: track 160.3 -> 239.1 mm, vias 12 -> 22
- net /In16/T8: track 0.00 -> 74.3 mm, vias 0 -> 1
- net /In16/T7: track 0.00 -> 71.8 mm, vias 0 -> 1
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Other:
- board text added: "19"
- board text added: "20"
- board text added: "21"
- board text added: "22"
- board text added: "23"
- board text added: "24"
- board text removed: "20V"
- board text removed: "20_IN"
- board text removed: "J5"
- board text removed: "WPC connector"
