File: IO_16x8_matrix/IO_16x8_matrix.kicad_pcb (KiCad board)
At the start: 2 copper layers, 97.6 x 67.3 mm, 211 parts, among them J1 Conn_01x06, J2 nmount SW Debug, J3 USB_C_Receptacle_USB2.0, J4 Conn_01x06, J5 Conn_01x09, J6 Conn_01x09, J7 Conn_01x09, J8 Conn_01x10, J9 Conn_01x10, Q1 MMBT3904, Q2 MMBT3904, Q3 MMBT3904, Q4 MMBT3904, Q5 MMBT3904, Q6 MMBT3904, Q7 MMBT3904, Q8 MMBT3904, SW1 Reset, SW2 Boot, SW3 ADDRESS, U1 ADM3483, U14 LMV321, U2 W25Q128JVSIQ, U3 RP2040, U4 SN74AHCT1G125, U5 AP2112K-3.3, U6 LM339, U7 LM339, U8 LM339, U9 LM339, Y1 12MHz,18pF

Commit message: opt routing
Parts:
- moved J6 31.6 mm to (190.7, 57.9), turned to -90 degrees
- moved J5 16.3 mm to (195.6, 66.3), turned to -90 degrees
- renumbered C32 to C25, C31 to C26, C30 to C27, C29 to C28, C28 to C29, C27 to C30, C26 to C31, C25 to C32, Q8 to Q1, Q7 to Q2, Q6 to Q3, Q5 to Q4, Q4 to Q5, Q3 to Q6, Q2 to Q7, Q1 to Q8, R31 to R20, R30 to R21, R29 to R22, R28 to R23, R35 to R24, R34 to R25, R33 to R26, R32 to R27, R23 to R28, R22 to R29, R21 to R30, R20 to R31, R27 to R32, R26 to R33, R25 to R34, R24 to R35
Connections:
- C25 pad 1: /Driver8/D8 -> /Driver8/D1
- C26 pad 1: /Driver8/D7 -> /Driver8/D2
- C27 pad 1: /Driver8/D6 -> /Driver8/D3
- C28 pad 1: /Driver8/D5 -> /Driver8/D4
- C29 pad 1: /Driver8/D4 -> /Driver8/D5
- C30 pad 1: /Driver8/D3 -> /Driver8/D6
- C31 pad 1: /Driver8/D2 -> /Driver8/D7
- C32 pad 1: /Driver8/D1 -> /Driver8/D8
- Q1 pad 3: /Driver8/D8 -> /Driver8/D1
- Q2 pad 3: /Driver8/D7 -> /Driver8/D2
- Q3 pad 3: /Driver8/D6 -> /Driver8/D3
- Q4 pad 3: /Driver8/D5 -> /Driver8/D4
- Q5 pad 3: /Driver8/D4 -> /Driver8/D5
- Q6 pad 3: /Driver8/D3 -> /Driver8/D6
- Q7 pad 3: /Driver8/D2 -> /Driver8/D7
- Q8 pad 3: /Driver8/D1 -> /Driver8/D8
- R20 pad 1: /Out_8 -> /Out_1
- R21 pad 1: /Out_7 -> /Out_2
- R22 pad 1: /Out_6 -> /Out_3
- R23 pad 1: /Out_5 -> /Out_4
- R24 pad 2: /Driver8/D8 -> /Driver8/D1
- R25 pad 2: /Driver8/D7 -> /Driver8/D2
- R26 pad 2: /Driver8/D6 -> /Driver8/D3
- R27 pad 2: /Driver8/D5 -> /Driver8/D4
- R28 pad 1: /Out_4 -> /Out_5
- R29 pad 1: /Out_3 -> /Out_6
- R30 pad 1: /Out_2 -> /Out_7
- R31 pad 1: /Out_1 -> /Out_8
- R32 pad 2: /Driver8/D4 -> /Driver8/D5
- R33 pad 2: /Driver8/D3 -> /Driver8/D6
- R34 pad 2: /Driver8/D2 -> /Driver8/D7
- R35 pad 2: /Driver8/D1 -> /Driver8/D8
- U3 pad 30: /Out_1 -> /Out_8
- U3 pad 31: /Out_2 -> /Out_7
- U3 pad 32: /Out_3 -> /Out_6
- U3 pad 34: /Out_4 -> /Out_5
- U3 pad 35: /Out_5 -> /Out_4
- U3 pad 36: /Out_6 -> /Out_3
- U3 pad 38: /Out_7 -> /Out_2
- U3 pad 39: /Out_8 -> /Out_1
Routing:
- net /Out_7: track 41.4 -> 56.7 mm
- net /Out_2: track 56.7 -> 41.4 mm
- net /Out_8: track 44.2 -> 53.5 mm
- net /Out_1: track 53.5 -> 44.2 mm
- net /Driver8/D2: track 27.6 -> 19.9 mm
- net /Out_6: track 44.8 -> 37.1 mm
- net /Out_3: track 37.1 -> 44.8 mm
- net /Driver8/D8: track 20.8 -> 13.9 mm
- net /Driver8/D1: track 19.3 -> 24.9 mm
- net (no net): track 4.72 -> 0.00 mm
- net /Out_5: track 42.7 -> 39.7 mm
- net /Out_4: track 39.7 -> 42.7 mm
- net /Driver8/D7: track 22.5 -> 24.7 mm
- net /Driver8/D5: track 19.9 -> 18.7 mm
- net /Driver8/D3: track 18.5 -> 19.4 mm
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Other:
- board text added: "IO_16x8_matrix"
- board text removed: "PPUC Out_8x10"

Commit message: prod_data
Other:
- rule pad_to_mask_clearance: 0 -> 0.05
Changed lines of the file:
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@@
   )
   (setup
-    (pad_to_mask_clearance 0)
+    (pad_to_mask_clearance 0.05)
     (pcbplotparams
       (layerselection 0x00010fc_ffffffff)
@@
       (drillshape 0)
       (scaleselection 1)
-      (outputdirectory "ProductionData/Gerber/")
+      (outputdirectory "ProductionData/")
     )
   )
@@
     (fp_line (start 33.28 -5.6) (end 33.28 5.15) (layer "F.Fab") (width 0.1))
     (fp_line (start -1.6 -5.6) (end 33.28 -5.6) (layer "F.Fab") (width 0.1))
-    (pad "1" thru_hole roundrect (at 0 0 270) (size 3.16 4.2) (drill 1.8) (layers *.Cu *.Mask) (roundrect_rratio 0.079114)
+    (pad "1" thru_hole roundrect (at 0 0 270) (size 3.16 4.2) (drill 1.8) (layers *.Cu *.Mask) (roundrect_rratio 0.07911392405)
       (net 27 "/Driver8/D1") (pinfunction "Pin_1") (pintype "passive"))
     (pad "2" thru_hole oval (at 3.96 0 270) (size 3.16 4.2) (drill 1.8) (layers *.Cu *.Mask)
@@
     (fp_line (start -1.6 -0.5) (end -0.892893 0) (layer "F.Fab") (width 0.1))
     (fp_line (start 37.24 5.15) (end -1.6 5.15) (layer "F.Fab") (width 0.1))
-    (pad "1" thru_hole roundrect (at 0 0 180) (size 3.16 4.2) (drill 1.8) (layers *.Cu *.Mask) (roundrect_rratio 0.079114)
+    (pad "1" thru_hole roundrect (at 0 0 180) (size 3.16 4.2) (drill 1.8) (layers *.Cu *.Mask) (roundrect_rratio 0.07911392405)
       (net 109 "/In16/T16") (pinfunction "Pin_1") (pintype "passive"))
     (pad "2" thru_hole oval (at 3.96 0 180) (size 3.16 4.2) (drill 1.8) (layers *.Cu *.Mask)
@@
     (fp_line (start 21.59 -2.92) (end -1.27 -2.92) (layer "F.Fab") (width 0.1))
     (fp_line (start -1.27 2.88) (end 21.59 2.88) (layer "F.Fab") (width 0.1))
-    (pad "1" thru_hole roundrect (at 0 0 270) (size 1.74 2.19) (drill 1.19) (layers *.Cu *.Mask) (roundrect_rratio 0.143678)
+    (pad "1" thru_hole roundrect (at 0 0 270) (size 1.74 2.19) (drill 1.19) (layers *.Cu *.Mask) (roundrect_rratio 0.1436781609)
       (net 27 "/Driver8/D1") (pinfunction "Pin_1") (pintype "passive"))
     (pad "2" thru_hole oval (at 2.54 0 270) (size 1.74 2.19) (drill 1.19) (layers *.Cu *.Mask)
@@
     (fp_line (start -1.6 -5.6) (end 37.24 -5.6) (layer "F.Fab") (width 0.1))
     (fp_line (start -1.6 -0.5) (end -0.892893 0) (layer "F.Fab") (width 0.1))
-    (pad "1" thru_hole roundrect (at 0 0 180) (size 3.16 4.2) (drill 1.8) (layers *.Cu *.Mask) (roundrect_rratio 0.079114)
+    (pad "1" thru_hole roundrect (at 0 0 180) (size 3.16 4.2) (drill 1.8) (layers *.Cu *.Mask) (roundrect_rratio 0.07911392405)
       (net 93 "/In16/T8") (pinfunction "Pin_1") (pintype "passive"))
     (pad "2" thru_hole oval (at 3.96 0 180) (size 3.16 4.2) (drill 1.8) (layers *.Cu *.Mask)
