File: IO_16x8_matrix/IO_16x8_matrix.kicad_pcb (KiCad board)
At the start: 2 copper layers, 97.6 x 67.3 mm, 211 parts, among them J1 Conn_01x06, J2 nmount SW Debug, J3 USB_C_Receptacle_USB2.0, J4 Conn_01x06, J5 Conn_01x09, J6 Conn_01x09, J7 Conn_01x09, J8 Conn_01x10, J9 Conn_01x10, Q1 MMBT3904, Q2 MMBT3904, Q3 MMBT3904, Q4 MMBT3904, Q5 MMBT3904, Q6 MMBT3904, Q7 MMBT3904, Q8 MMBT3904, SW1 Reset, SW2 Boot, SW3 ADDRESS, U1 ADM3483, U14 LMV321, U2 W25Q128JVSIQ, U3 RP2040, U4 SN74AHCT1G125, U5 AP2112K-3.3, U6 LM339, U7 LM339, U8 LM339, U9 LM339, Y1 12MHz,18pF

Commit message: V1.0.0
Parts:
- removed F1: T500mA,<0.3Ω, Fuse:Fuse_1206_3216Metric
- removed R3, R5: 1k, Resistor_SMD:R_0402_1005Metric
- added D23: 1A, Diode_SMD:D_SOD-323, F.Cu at (169.5, 60.1)
- added JP1: Jumper_2_Open, Connector_PinHeader_2.54mm:PinHeader_1x02_P2.54mm_Vertical, F.Cu at (141.7, 55.5)
Connections:
- J1 pad 4: GND -> /A
- J1 pad 5: GND -> /B
- R4 pad 1: /A -> Net-(R4-Pad1)
Routing:
- net /A: track 27.0 -> 49.2 mm
- net /B: track 27.8 -> 45.0 mm
- net GND: track 407.9 -> 397.9 mm
- net Net-(R4-Pad1): track 0.00 -> 6.97 mm
- net +5V: track 297.3 -> 294.1 mm
- net /5V_IN: track 38.2 -> 39.0 mm
