File: IO_16x8_matrix/IO_16x8_matrix.kicad_sch (KiCad schematic)
At the start: 76 parts, among them J1 Conn_01x06, J2 nmount SW Debug, J3 USB_C_Receptacle_USB2.0, J4 Conn_01x06, SW1 Reset, SW2 Boot, SW3 ADDRESS, U1 ADM3483, U14 LMV321, U2 W25Q128JVSIQ, U3 RP2040, U4 SN74AHCT1G125, U5 AP2112K-3.3, Y1 12MHz,18pF

Commit message: opt routing
Connections:
- net Out_1: now also U3.39 (GPIO27_ADC1); no longer U3.30 (GPIO19)
- net Out_2: now also U3.38 (GPIO26_ADC0); no longer U3.31 (GPIO20)
- net Out_3: now also U3.36 (GPIO24); no longer U3.32 (GPIO21)
- net Out_4: now also U3.35 (GPIO23); no longer U3.34 (GPIO22)
- net Out_5: now also U3.34 (GPIO22); no longer U3.35 (GPIO23)
- net Out_6: now also U3.32 (GPIO21); no longer U3.36 (GPIO24)
- net Out_7: now also U3.31 (GPIO20); no longer U3.38 (GPIO26_ADC0)
- net Out_8: now also U3.30 (GPIO19); no longer U3.39 (GPIO27_ADC1)
