File: IO_16x8_matrix/IO_16x8_matrix.kicad_sch (KiCad schematic)
At the start: 76 parts, among them J1 Conn_01x06, J2 nmount SW Debug, J3 USB_C_Receptacle_USB2.0, J4 Conn_01x06, SW1 Reset, SW2 Boot, SW3 ADDRESS, U1 ADM3483, U14 LMV321, U2 W25Q128JVSIQ, U3 RP2040, U4 SN74AHCT1G125, U5 AP2112K-3.3, Y1 12MHz,18pF

Commit message: V1.0.0
Parts:
- removed F1: T500mA,<0.3Ω, Fuse:Fuse_1206_3216Metric, symbol Device:Fuse
- removed R3, R5: 1k, Resistor_SMD:R_0402_1005Metric, symbol Device:R
- added D23: 1A, Diode_SMD:D_SOD-323, symbol Device:D_Schottky
- added JP1: Jumper_2_Open, Connector_PinHeader_2.54mm:PinHeader_1x02_P2.54mm_Vertical, symbol Jumper:Jumper_2_Open
- C22: JLCPCB Rotation Offset (none) -> 180
- SW3, U5: JLCPCB Rotation Offset (none) -> 90
- TP4, TP5: now left out of the parts list
- U3: JLCPCB Rotation Offset (none) -> -90
Connections:
- net +5V: now also D23.1 (K)
- net 5V_IN: now also D23.2 (A)
- net A: now also J1.4 (Pin_4), JP1.2 (B); no longer R4.1
- net B: now also J1.5 (Pin_5)
- net GND: no longer J1.4 (Pin_4), J1.5 (Pin_5)
- new net: JP1.1 (A), R4.1
Other:
- moved on the sheet: D1
