File: IO_16x8_matrix/rtn_sub_4x.kicad_sch (KiCad schematic)
At the start: 23 parts, among them U6 LM339

Commit message: routed
Parts:
- U6: footprint (none) -> Package_SO:SOIC-14_3.9x8.7mm_P1.27mm
Changed lines of the file:
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@@
     (property "Reference" "U6" (id 0) (at 185.42 43.18 0))
     (property "Value" "LM339" (id 1) (at 185.42 45.72 0))
-    (property "Footprint" "" (id 2) (at 186.69 55.88 0)
+    (property "Footprint" "Package_SO:SOIC-14_3.9x8.7mm_P1.27mm" (id 2) (at 186.69 55.88 0)
       (effects (font (size 1.27 1.27)) hide)
     )
@@
     (property "Reference" "U6" (id 0) (at 185.42 92.71 0))
     (property "Value" "LM339" (id 1) (at 185.42 95.25 0))
-    (property "Footprint" "" (id 2) (at 186.69 105.41 0)
+    (property "Footprint" "Package_SO:SOIC-14_3.9x8.7mm_P1.27mm" (id 2) (at 186.69 105.41 0)
       (effects (font (size 1.27 1.27)) hide)
     )
@@
     (property "Reference" "U6" (id 0) (at 81.28 43.18 0))
     (property "Value" "LM339" (id 1) (at 81.28 45.72 0))
-    (property "Footprint" "" (id 2) (at 82.55 55.88 0)
+    (property "Footprint" "Package_SO:SOIC-14_3.9x8.7mm_P1.27mm" (id 2) (at 82.55 55.88 0)
       (effects (font (size 1.27 1.27)) hide)
     )
@@
     (property "Reference" "U6" (id 0) (at 81.28 92.71 0))
     (property "Value" "LM339" (id 1) (at 81.28 95.25 0))
-    (property "Footprint" "" (id 2) (at 82.55 105.41 0)
+    (property "Footprint" "Package_SO:SOIC-14_3.9x8.7mm_P1.27mm" (id 2) (at 82.55 105.41 0)
       (effects (font (size 1.27 1.27)) hide)
     )
@@
       (effects (font (size 1.27 1.27)) (justify left))
     )
-    (property "Footprint" "" (id 2) (at 82.55 160.02 0)
-      (effects (font (size 1.27 1.27)) hide)
-    )
+    (property "Footprint" "Package_SO:SOIC-14_3.9x8.7mm_P1.27mm" (id 2) (at 82.55 160.02 0)
+      (effects (font (size 1.27 1.27)) hide)
+    )
